File: output_stage.kicad_sch (KiCad schematic)
At the start: 26 parts, among them J2 XLR3, U7 OPA1612AxD, U8 OPA1612AxD

Commit message: traced o/s
Parts:
- removed J2: XLR3, Connector_Audio:Jack_XLR_Neutrik_NC3MAH_Horizontal, symbol Connector_Audio:XLR3
- added J5: XLR_L, Connector_Audio:Jack_XLR_Neutrik_NC3MAH-0_Horizontal, symbol Connector_Audio:XLR3_Ground
Connections:
- net GNDA: now also J5.1, J5.G
- net OUT_Lb: now reaches C30.1, R26.1
- net OUT_Lb: now also J5.2
- net OUT_L: now reaches C29.1, R27.1
- net OUT_L: now also J5.3
Changed lines of the file:
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@@
 	)
 	(junction
-		(at 148.59 41.91)
-		(diameter 0)
-		(color 0 0 0 0)
-	)
-	(junction
 		(at 83.82 113.03)
 		(diameter 0)
@@
 	)
 	(junction
+		(at 161.29 55.88)
+		(diameter 0)
+		(color 0 0 0 0)
+	)
+	(junction
 		(at 83.82 36.83)
 		(diameter 0)
@@
 	)
 	(junction
+		(at 148.59 41.91)
+		(diameter 0)
+		(color 0 0 0 0)
+	)
+	(junction
 		(at 54.61 36.83)
 		(diameter 0)
@@
 	(wire
 		(pts
-			(xy 153.67 63.5) (xy 153.67 41.91)
+			(xy 54.61 30.48) (xy 67.31 30.48)
 		)
 		(stroke
@@
 	(wire
 		(pts
-			(xy 54.61 30.48) (xy 67.31 30.48)
+			(xy 254 31.75) (xy 260.35 31.75)
 		)
 		(stroke
@@
 	(wire
 		(pts
-			(xy 254 31.75) (xy 260.35 31.75)
+			(xy 101.6 48.26) (xy 109.22 48.26)
 		)
 		(stroke
@@
 	(wire
 		(pts
-			(xy 101.6 48.26) (xy 109.22 48.26)
+			(xy 153.67 60.96) (xy 153.67 55.88)
 		)
 		(stroke
@@
 	(wire
 		(pts
+			(xy 152.4 41.91) (xy 152.4 63.5)
+		)
+		(stroke
+			(width 0)
+			(type default)
+		)
+	)
+	(wire
+		(pts
 			(xy 30.48 54.61) (xy 39.37 54.61)
 		)
@@
 	(wire
 		(pts
+			(xy 153.67 63.5) (xy 152.4 63.5)
+		)
+		(stroke
+			(width 0)
+			(type default)
+		)
+	)
+	(wire
+		(pts
 			(xy 254 46.99) (xy 260.35 46.99)
 		)
@@
 	(wire
 		(pts
+			(xy 153.67 55.88) (xy 161.29 55.88)
+		)
+		(stroke
+			(width 0)
+			(type default)
+		)
+	)
+	(wire
+		(pts
 			(xy 72.39 113.03) (xy 83.82 113.03)
 		)
@@
 	(wire
 		(pts
-			(xy 148.59 41.91) (xy 153.67 41.91)
+			(xy 148.59 41.91) (xy 152.4 41.91)
 		)
 		(stroke
@@
 		)
 	)
+	(global_label "OUT_L"
+		(shape input)
+		(at 152.4 41.91 0)
+		(fields_autoplaced yes)
+		(effects
+			(font
+				(size 1.27 1.27)
+			)
+			(justify left)
+		)
+		(property "Intersheetrefs" "${INTERSHEET_REFS}"
+			(at 161.0095 41.91 0)
+			(hide yes)
+			(show_name no)
+			(do_not_autoplace no)
+			(effects
+				(font
+					(size 1.27 1.27)
+				)
+				(justify left)
+			)
+		)
+	)
+	(global_label "OUT_Lb"
+		(shape input)
+		(at 161.29 92.71 0)
+		(fields_autoplaced yes)
+		(effects
+			(font
+				(size 1.27 1.27)
+			)
+			(justify left)
+		)
+		(property "Intersheetrefs" "${INTERSHEET_REFS}"
+			(at 171.0485 92.71 0)
+			(hide yes)
+			(show_name no)
+			(do_not_autoplace no)
+			(effects
+				(font
+					(size 1.27 1.27)
+				)
+				(justify left)
+			)
+		)
+	)
 	(global_label "DAC1B"
 		(shape input)
@@
 	)
 	(symbol
-		(lib_id "Connector_Audio:XLR3")
-		(at 161.29 63.5 270)
-		(unit 1)
-		(body_style 1)
-		(exclude_from_sim no)
-		(in_bom yes)
-		(on_board yes)
-		(in_pos_files yes)
-		(dnp no)
-		(fields_autoplaced yes)
-		(property "Reference" "J2"
-			(at 167.64 62.2299 90)
-			(show_name no)
-			(do_not_autoplace no)
-			(effects
-				(font
-					(size 1.27 1.27)
-				)
-				(justify left)
-			)
-		)
-		(property "Value" "XLR3"
-			(at 167.64 64.7699 90)
-			(show_name no)
-			(do_not_autoplace no)
-			(effects
-				(font
-					(size 1.27 1.27)
-				)
-				(justify left)
-			)
-		)
-		(property "Footprint" "Connector_Audio:Jack_XLR_Neutrik_NC3MAH_Horizontal"
-			(at 161.29 63.5 0)
-			(hide yes)
-			(show_name no)
-			(do_not_autoplace no)
-			(effects
-				(font
-					(size 1.27 1.27)
-				)
-			)
-		)
-		(property "Datasheet" ""
-			(at 161.29 63.5 0)
-			(hide yes)
-			(show_name no)
-			(do_not_autoplace no)
-			(effects
-				(font
-					(size 1.27 1.27)
-				)
-			)
-		)
-		(property "Description" "XLR Connector, Male or Female, 3 Pins"
-			(at 161.29 63.5 0)
-			(hide yes)
-			(show_name no)
-			(do_not_autoplace no)
-			(effects
-				(font
-					(size 1.27 1.27)
-				)
-			)
-		)
-		(pin "2"
-		)
-		(pin "3"
-		)
-		(pin "1"
-		)
-		(instances
-			(project "es9039_dac"
-				(path "/47c411d8-44e2-450d-908b-0e7677743dac"
-					(reference "J2")
-					(unit 1)
-				)
-			)
-		)
-	)
-	(symbol
 		(lib_id "power:GNDA")
 		(at 173.99 55.88 0)
@@
 					(unit 1)
 				)
+			)
+		)
+	)
+	(symbol
+		(lib_id "Connector_Audio:XLR3_Ground")
+		(at 161.29 63.5 270)
+		(unit 1)
+		(body_style 1)
+		(exclude_from_sim no)
+		(in_bom yes)
+		(on_board yes)
+		(in_pos_files yes)
+		(dnp no)
+		(fields_autoplaced yes)
+		(property "Reference" "J5"
+			(at 167.64 62.2299 90)
+			(show_name no)
+			(do_not_autoplace no)
+			(effects
+				(font
+					(size 1.27 1.27)
+				)
+				(justify left)
+			)
+		)
+		(property "Value" "XLR_L"
+			(at 167.64 64.7699 90)
+			(show_name no)
+			(do_not_autoplace no)
+			(effects
+				(font
+					(size 1.27 1.27)
+				)
+				(justify left)
+			)
+		)
+		(property "Footprint" "Connector_Audio:Jack_XLR_Neutrik_NC3MAH-0_Horizontal"
+			(at 161.29 63.5 0)
+			(hide yes)
+			(show_name no)
+			(do_not_autoplace no)
+			(effects
+				(font
+					(size 1.27 1.27)
+				)
+			)
+		)
+		(property "Datasheet" ""
+			(at 161.29 63.5 0)
+			(hide yes)
+			(show_name no)
+			(do_not_autoplace no)
+			(effects
+				(font
+					(size 1.27 1.27)
+				)
+			)
+		)
+		(property "Description" "XLR Connector, Male or Female, 3 Pins, Discrete Ground Pin"
+			(at 161.29 63.5 0)
+			(hide yes)
+			(show_name no)
+			(do_not_autoplace no)
+			(effects
+				(font
+					(size 1.27 1.27)
+				)
+			)
+		)
+		(pin "3"
+		)
+		(pin "G"
+		)
+		(pin "2"
+		)
+		(pin "1"
+		)
+		(instances
+			(project "es9039_dac"
+				(path "/47c411d8-44e2-450d-908b-0e7677743dac"
+					(reference "J5")
+					(unit 1)
+				)
