File: output_stage2.kicad_sch (KiCad schematic)
At the start: 24 parts, among them J3 XLR3, U8 OPA1612AxD, U9 OPA1612AxD

Commit message: traced o/s
Parts:
- removed J3: XLR3, Connector_Audio:Jack_XLR_Neutrik_NC3MAH_Horizontal, symbol Connector_Audio:XLR3
- added J3: XLR_R, Connector_Audio:Jack_XLR_Neutrik_NC3MAH-0_Horizontal, symbol Connector_Audio:XLR3_Ground
Connections:
- net GNDA: now also J3.1, J3.G
- net OUT_R: now reaches C38.1, R39.1
- net OUT_R: now also J3.3
- net OUT_Rb: now reaches C39.1, R40.1
- net OUT_Rb: now also J3.2
Changed lines of the file:
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@@
 	)
 	(junction
+		(at 172.72 69.85)
+		(diameter 0)
+		(color 0 0 0 0)
+	)
+	(junction
 		(at 143.51 55.88)
 		(diameter 0)
@@
 	(wire
 		(pts
+			(xy 165.1 77.47) (xy 163.83 77.47)
+		)
+		(stroke
+			(width 0)
+			(type default)
+		)
+	)
+	(wire
+		(pts
 			(xy 97.79 71.12) (xy 95.25 71.12)
 		)
@@
 	(wire
 		(pts
+			(xy 163.83 55.88) (xy 163.83 77.47)
+		)
+		(stroke
+			(width 0)
+			(type default)
+		)
+	)
+	(wire
+		(pts
 			(xy 160.02 106.68) (xy 172.72 106.68)
 		)
@@
 	(wire
 		(pts
-			(xy 165.1 77.47) (xy 165.1 55.88)
-		)
-		(stroke
-			(width 0)
-			(type default)
-		)
-	)
-	(wire
-		(pts
 			(xy 95.25 120.65) (xy 95.25 106.68)
 		)
@@
 	(wire
 		(pts
-			(xy 160.02 55.88) (xy 165.1 55.88)
+			(xy 160.02 55.88) (xy 163.83 55.88)
 		)
 		(stroke
@@
 	(wire
 		(pts
+			(xy 165.1 74.93) (xy 165.1 69.85)
+		)
+		(stroke
+			(width 0)
+			(type default)
+		)
+	)
+	(wire
+		(pts
 			(xy 143.51 106.68) (xy 151.13 106.68)
 		)
@@
 	(wire
 		(pts
+			(xy 165.1 69.85) (xy 172.72 69.85)
+		)
+		(stroke
+			(width 0)
+			(type default)
+		)
+	)
+	(wire
+		(pts
 			(xy 95.25 44.45) (xy 95.25 50.8)
 		)
@@
 		)
 	)
+	(global_label "OUT_Rb"
+		(shape input)
+		(at 172.72 106.68 0)
+		(fields_autoplaced yes)
+		(effects
+			(font
+				(size 1.27 1.27)
+			)
+			(justify left)
+		)
+		(property "Intersheetrefs" "${INTERSHEET_REFS}"
+			(at 182.7204 106.68 0)
+			(hide yes)
+			(show_name no)
+			(do_not_autoplace no)
+			(effects
+				(font
+					(size 1.27 1.27)
+				)
+				(justify left)
+			)
+		)
+	)
+	(global_label "OUT_R"
+		(shape input)
+		(at 163.83 55.88 0)
+		(fields_autoplaced yes)
+		(effects
+			(font
+				(size 1.27 1.27)
+			)
+			(justify left)
+		)
+		(property "Intersheetrefs" "${INTERSHEET_REFS}"
+			(at 172.6814 55.88 0)
+			(hide yes)
+			(show_name no)
+			(do_not_autoplace no)
+			(effects
+				(font
+					(size 1.27 1.27)
+				)
+				(justify left)
+			)
+		)
+	)
 	(symbol
 		(lib_id "Device:R_Small")
@@
 	)
 	(symbol
-		(lib_id "power:GNDA")
-		(at 185.42 69.85 0)
+		(lib_id "Connector_Audio:XLR3_Ground")
+		(at 172.72 77.47 270)
 		(unit 1)
 		(body_style 1)
@@
 		(in_pos_files yes)
 		(dnp no)
-		(property "Reference" "#PWR056"
-			(at 185.42 76.2 0)
-			(hide yes)
+		(fields_autoplaced yes)
+		(property "Reference" "J3"
+			(at 179.07 76.1999 90)
 			(show_name no)
 			(do_not_autoplace no)
@@
 					(size 1.27 1.27)
 				)
+				(justify left)
 			)
 		)
-		(property "Value" "GNDA"
-			(at 185.42 73.914 0)
+		(property "Value" "XLR_R"
+			(at 179.07 78.7399 90)
 			(show_name no)
 			(do_not_autoplace no)
@@
 					(size 1.27 1.27)
 				)
+				(justify left)
 			)
 		)
-		(property "Footprint" ""
-			(at 185.42 69.85 0)
+		(property "Footprint" "Connector_Audio:Jack_XLR_Neutrik_NC3MAH-0_Horizontal"
+			(at 172.72 77.47 0)
 			(hide yes)
 			(show_name no)
@@
 		)
 		(property "Datasheet" ""
-			(at 185.42 69.85 0)
+			(at 172.72 77.47 0)
 			(hide yes)
 			(show_name no)
@@
 			)
 		)
-		(property "Description" "Power symbol creates a global label with name \"GNDA\" , analog ground"
-			(at 185.42 69.85 0)
+		(property "Description" "XLR Connector, Male or Female, 3 Pins, Discrete Ground Pin"
+			(at 172.72 77.47 0)
 			(hide yes)
 			(show_name no)
@@
 			)
 		)
+		(pin "3"
+		)
+		(pin "G"
+		)
+		(pin "2"
+		)
 		(pin "1"
 		)
@@
 			(project "es9039_dac"
 				(path "/bdbdcc8c-b268-4bd9-89c9-eead5f36a92c"
-					(reference "#PWR056")
+					(reference "J3")
 					(unit 1)
 				)
@@
 	)
 	(symbol
-		(lib_id "Connector_Audio:XLR3")
-		(at 172.72 77.47 270)
+		(lib_id "power:GNDA")
+		(at 185.42 69.85 0)
 		(unit 1)
 		(body_style 1)
@@
 		(in_pos_files yes)
 		(dnp no)
-		(fields_autoplaced yes)
-		(property "Reference" "J3"
-			(at 179.07 76.1999 90)
+		(property "Reference" "#PWR056"
+			(at 185.42 76.2 0)
+			(hide yes)
 			(show_name no)
 			(do_not_autoplace no)
@@
 					(size 1.27 1.27)
 				)
-				(justify left)
 			)
 		)
-		(property "Value" "XLR3"
-			(at 179.07 78.7399 90)
+		(property "Value" "GNDA"
+			(at 185.42 73.914 0)
 			(show_name no)
 			(do_not_autoplace no)
@@
 					(size 1.27 1.27)
 				)
-				(justify left)
 			)
 		)
-		(property "Footprint" "Connector_Audio:Jack_XLR_Neutrik_NC3MAH_Horizontal"
-			(at 172.72 77.47 0)
+		(property "Footprint" ""
+			(at 185.42 69.85 0)
 			(hide yes)
 			(show_name no)
@@
 		)
 		(property "Datasheet" ""
-			(at 172.72 77.47 0)
+			(at 185.42 69.85 0)
 			(hide yes)
 			(show_name no)
@@
 			)
 		)
-		(property "Description" "XLR Connector, Male or Female, 3 Pins"
-			(at 172.72 77.47 0)
+		(property "Description" "Power symbol creates a global label with name \"GNDA\" , analog ground"
+			(at 185.42 69.85 0)
 			(hide yes)
 			(show_name no)
@@
 			)
 		)
-		(pin "2"
-		)
-		(pin "3"
-		)
 		(pin "1"
 		)
@@
 			(project "es9039_dac"
 				(path "/bdbdcc8c-b268-4bd9-89c9-eead5f36a92c"
-					(reference "J3")
+					(reference "#PWR056")
 					(unit 1)
 				)
